Commit message: Change dae to obj

File: pal_robotics/tiago_dual_description/urdf/tiago_dual.urdf (robot description, URDF)
Before this commit: robot tiago_dual, 69 links, 68 joints
Links:
- link arm_left_1_link: geometry collision mesh filename=package://tiago_dual_description/urdf/tiago_dual/stl/arm_1_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 scale=1.0 -1.0 -1.0; visual mesh filename=package://tiago_dual_description/urdf/tiago_dual/obj/arm_1.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 scale=1.0 -1.0 -1.0
- link arm_left_2_link: geometry collision mesh filename=package://tiago_dual_description/urdf/tiago_dual/stl/arm_2_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 scale=1.0 1.0 -1.0; visual mesh filename=package://tiago_dual_description/urdf/tiago_dual/obj/arm_2.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 scale=1.0 1.0 -1.0
- link arm_left_3_link: geometry collision mesh filename=package://tiago_dual_description/urdf/tiago_dual/stl/arm_3_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 scale=1.0 1.0 -1.0; visual mesh filename=package://tiago_dual_description/urdf/tiago_dual/obj/arm_3.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 scale=1.0 1.0 -1.0
- link arm_left_4_link: geometry collision mesh filename=package://tiago_dual_description/urdf/tiago_dual/stl/arm_4_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 scale=-1.0 -1.0 -1.0; visual mesh filename=package://tiago_dual_description/urdf/tiago_dual/obj/arm_4.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 scale=-1.0 -1.0 -1.0
- link arm_left_5_link: geometry collision mesh filename=package://tiago_dual_description/urdf/tiago_dual/stl/arm_5_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 scale=-1.0 -1.0 -1.0; visual mesh filename=package://tiago_dual_description/urdf/tiago_dual/obj/arm_5-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 scale=-1.0 -1.0 -1.0
- link arm_left_6_link: geometry collision mesh filename=package://tiago_dual_description/urdf/tiago_dual/stl/arm_6_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 scale=-1.0 1.0 1.0; visual mesh filename=package://tiago_dual_description/urdf/tiago_dual/obj/arm_6-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 scale=-1.0 1.0 1.0
- link arm_left_7_link: mass 0.100 -> 0.1
- link arm_right_1_link: geometry collision mesh filename=package://tiago_dual_description/urdf/tiago_dual/stl/arm_1_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 scale=1.0 -1.0 1.0; visual mesh filename=package://tiago_dual_description/urdf/tiago_dual/obj/arm_1.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 scale=1.0 -1.0 1.0
- link arm_right_2_link: geometry collision mesh filename=package://tiago_dual_description/urdf/tiago_dual/stl/arm_2_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 scale=1.0 1.0 1.0; visual mesh filename=package://tiago_dual_description/urdf/tiago_dual/obj/arm_2.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 scale=1.0 1.0 1.0
- link arm_right_3_link: geometry collision mesh filename=package://tiago_dual_description/urdf/tiago_dual/stl/arm_3_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 scale=1.0 1.0 1.0; visual mesh filename=package://tiago_dual_description/urdf/tiago_dual/obj/arm_3.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 scale=1.0 1.0 1.0
- link arm_right_4_link: geometry collision mesh filename=package://tiago_dual_description/urdf/tiago_dual/stl/arm_4_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 scale=1.0 1.0 1.0; visual mesh filename=package://tiago_dual_description/urdf/tiago_dual/obj/arm_4.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 scale=1.0 1.0 1.0
- link arm_right_5_link: geometry collision mesh filename=package://tiago_dual_description/urdf/tiago_dual/stl/arm_5_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 scale=1.0 1.0 1.0; visual mesh filename=package://tiago_dual_description/urdf/tiago_dual/obj/arm_5-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 scale=1.0 1.0 1.0
- link arm_right_6_link: geometry collision mesh filename=package://tiago_dual_description/urdf/tiago_dual/stl/arm_6_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 scale=1.0 1.0 1.0; visual mesh filename=package://tiago_dual_description/urdf/tiago_dual/obj/arm_6-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 scale=1.0 1.0 1.0
- link arm_right_7_link: mass 0.100 -> 0.1
- link base_antenna_left_link: mass 0.000001 -> 1e-06; geometry collision cylinder length=0.17 radius=0.005; visual mesh filename=package://tiago_dual_description/urdf/tiago_dual/obj/antenn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
- link base_antenna_right_link: mass 0.000001 -> 1e-06; geometry collision cylinder length=0.17 radius=0.005; visual mesh filename=package://tiago_dual_description/urdf/tiago_dual/obj/antenn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
- link base_cover_link: mass 0.25821000000 -> 0.25821; geometry visual mesh filename=package://tiago_dual_description/urdf/tiago_dual/obj/base_r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
- link base_laser_link: mass 0.28922000000 -> 0.28922; geometry visual mesh filename=package://tiago_dual_description/urdf/tiago_dual/obj/sick_t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
- link base_link: geometry collision mesh filename=package://tiago_dual_description/urdf/tiago_dual/stl/base_c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; visual mesh filename=package://tiago_dual_description/urdf/tiago_dual/obj/base.o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
- link base_sonar_01_link: geometry visual mesh filename=package://tiago_dual_description/urdf/tiago_dual/obj/srf05.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
- link base_sonar_02_link: geometry visual mesh filename=package://tiago_dual_description/urdf/tiago_dual/obj/srf05.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
- link base_sonar_03_link: geometry visual mesh filename=package://tiago_dual_description/urdf/tiago_dual/obj/srf05.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
- link caster_back_left_1_link: geometry visual mesh filename=package://tiago_dual_description/urdf/tiago_dual/obj/caster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
- link caster_back_left_2_link: geometry collision sphere radius=0.025; visual mesh filename=package://tiago_dual_description/urdf/tiago_dual/obj/caster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
- link caster_back_right_1_link: geometry visual mesh filename=package://tiago_dual_description/urdf/tiago_dual/obj/caster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
- link caster_back_right_2_link: geometry collision sphere radius=0.025; visual mesh filename=package://tiago_dual_description/urdf/tiago_dual/obj/caster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
- link caster_front_left_1_link: geometry visual mesh filename=package://tiago_dual_description/urdf/tiago_dual/obj/caster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
- link caster_front_left_2_link: geometry collision sphere radius=0.025; visual mesh filename=package://tiago_dual_description/urdf/tiago_dual/obj/caster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
- link caster_front_right_1_link: geometry visual mesh filename=package://tiago_dual_description/urdf/tiago_dual/obj/caster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
- link caster_front_right_2_link: geometry collision sphere radius=0.025; visual mesh filename=package://tiago_dual_description/urdf/tiago_dual/obj/caster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
- link gripper_left_left_finger_link: mass 0.109980 -> 0.10998; geometry collision box size=0.01 0.05 0.11; visual mesh filename=package://tiago_dual_description/urdf/tiago_dual/obj/grippe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
- link gripper_left_link: mass 0.602660 -> 0.60266; geometry collision mesh filename=package://tiago_dual_description/urdf/tiago_dual/stl/grippe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; visual mesh filename=package://tiago_dual_description/urdf/tiago_dual/obj/grippe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
- link gripper_left_right_finger_link: mass 0.109980 -> 0.10998; geometry collision box size=0.01 0.05 0.11; visual mesh filename=package://tiago_dual_description/urdf/tiago_dual/obj/grippe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 scale=-1.0 -1.0 1.0
- link gripper_right_left_finger_link: mass 0.109980 -> 0.10998; geometry collision box size=0.01 0.05 0.11; visual mesh filename=package://tiago_dual_description/urdf/tiago_dual/obj/grippe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
- link gripper_right_link: mass 0.602660 -> 0.60266; geometry collision mesh filename=package://tiago_dual_description/urdf/tiago_dual/stl/grippe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; visual mesh filename=package://tiago_dual_description/urdf/tiago_dual/obj/grippe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
- link gripper_right_right_finger_link: mass 0.109980 -> 0.10998; geometry collision box size=0.01 0.05 0.11; visual mesh filename=package://tiago_dual_description/urdf/tiago_dual/obj/grippe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 scale=-1.0 -1.0 1.0
- link head_1_link: mass 0.62220 -> 0.6222; geometry collision mesh filename=package://tiago_dual_description/urdf/tiago_dual/stl/head_1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 scale=1.0 1.0 1.0; visual mesh filename=package://tiago_dual_description/urdf/tiago_dual/obj/head_1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 scale=1.0 1.0 1.0
- link head_2_link: geometry collision mesh filename=package://tiago_dual_description/urdf/tiago_dual/stl/head_2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 scale=1.0 1.0 1.0; visual mesh filename=package://tiago_dual_description/urdf/tiago_dual/obj/head_2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 scale=1.0 1.0 1.0
- link suspension_left_link: mass 10 -> 10.0
- link suspension_right_link: mass 10 -> 10.0
- link torso_fixed_link: mass 14.01360 -> 14.0136; geometry collision box size=0.25 0.25 0.1; collision box size=0.4 0.25 0.04
- link torso_lift_link: geometry collision mesh filename=package://tiago_dual_description/urdf/tiago_dual/stl/torso_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 scale=1.0 1.0 1.0; collision mesh filename=package://tiago_dual_description/urdf/tiago_dual/stl/torso_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 scale=1.0 1.0 1.0
- link wheel_left_link: geometry collision sphere radius=0.0985; visual mesh filename=package://tiago_dual_description/urdf/tiago_dual/obj/wheel.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
- link wheel_right_link: geometry collision sphere radius=0.0985; visual mesh filename=package://tiago_dual_description/urdf/tiago_dual/obj/wheel.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
- link xtion_link: mass 0.21970000000 -> 0.2197
Joints:
- joint arm_left_1_joint: axis 0 0 1 -> 0.0 0.0 1.0; origin xyz=0.02556 0.19 -0.171 rpy=3.141592653589793 0 1.5707963267948966 -> xyz=0.02556 0.19 -0.171 rpy=3.141592653589793 0.0 1.5707963267948966
- joint arm_left_2_joint: axis 0 0 1 -> 0.0 0.0 1.0
- joint arm_left_3_joint: axis 0 0 1 -> 0.0 0.0 1.0; limit lower=-0.7853981633974483 upper=3.9269908169872414 effort=26 velocity=2.35 -> lower=-0.7853981633974483 upper=3.9269908169872414 effort=26.0 velocity=2.35
- joint arm_left_4_joint: axis 0 0 1 -> 0.0 0.0 1.0; limit lower=-0.39269908169872414 upper=2.356194490192345 effort=26 velocity=2.35 -> lower=-0.39269908169872414 upper=2.356194490192345 effort=26.0 velocity=2.35
- joint arm_left_5_joint: axis 0 0 1 -> 0.0 0.0 1.0; limit lower=-2.0943951023931953 upper=2.0943951023931953 effort=3 velocity=1.95 -> lower=-2.0943951023931953 upper=2.0943951023931953 effort=3.0 velocity=1.95
- joint arm_left_6_joint: axis 0 0 1 -> 0.0 0.0 1.0; origin xyz=0 0 -0.15 rpy=0.0 -1.5707963267948966 -1.5707963267948966 -> xyz=0.0 0.0 -0.15 rpy=0.0 -1.5707963267948966 -1.5707963267948966
- joint arm_left_7_joint: axis 0 0 1 -> 0.0 0.0 1.0; origin xyz=0 0 0 rpy=1.5707963267948966 0.0 1.5707963267948966 -> xyz=0.0 0.0 0.0 rpy=1.5707963267948966 0.0 1.5707963267948966
- joint arm_left_tool_joint: origin xyz=0 0 -0.046 rpy=1.5707963267948966 1.5707963267948966 3.141592653589793 -> xyz=0.0 0.0 -0.046 rpy=1.5707963267948966 1.5707963267948966 3.141592653589793
- joint arm_right_1_joint: axis 0 0 1 -> 0.0 0.0 1.0; origin xyz=0.02556 -0.19 -0.171 rpy=0 0 -1.5707963267948966 -> xyz=0.02556 -0.19 -0.171 rpy=0.0 0.0 -1.5707963267948966
- joint arm_right_2_joint: axis 0 0 1 -> 0.0 0.0 1.0
- joint arm_right_3_joint: axis 0 0 1 -> 0.0 0.0 1.0; limit lower=-0.7853981633974483 upper=3.9269908169872414 effort=26 velocity=2.35 -> lower=-0.7853981633974483 upper=3.9269908169872414 effort=26.0 velocity=2.35
- joint arm_right_4_joint: axis 0 0 1 -> 0.0 0.0 1.0; limit lower=-0.39269908169872414 upper=2.356194490192345 effort=26 velocity=2.35 -> lower=-0.39269908169872414 upper=2.356194490192345 effort=26.0 velocity=2.35
- joint arm_right_5_joint: axis 0 0 1 -> 0.0 0.0 1.0; limit lower=-2.0943951023931953 upper=2.0943951023931953 effort=3 velocity=1.95 -> lower=-2.0943951023931953 upper=2.0943951023931953 effort=3.0 velocity=1.95
- joint arm_right_6_joint: axis 0 0 1 -> 0.0 0.0 1.0; origin xyz=0 0 0.15 rpy=0.0 -1.5707963267948966 -1.5707963267948966 -> xyz=0.0 0.0 0.15 rpy=0.0 -1.5707963267948966 -1.5707963267948966
- joint arm_right_7_joint: axis 0 0 1 -> 0.0 0.0 1.0; origin xyz=0 0 0 rpy=1.5707963267948966 0.0 1.5707963267948966 -> xyz=0.0 0.0 0.0 rpy=1.5707963267948966 0.0 1.5707963267948966
- joint arm_right_tool_joint: origin xyz=0 0 0.046 rpy=1.5707963267948966 -1.5707963267948966 3.141592653589793 -> xyz=0.0 0.0 0.046 rpy=1.5707963267948966 -1.5707963267948966 3.141592653589793
- joint base_antenna_left_joint: origin xyz=-0.201 0.1062 0.195 rpy=0 0 0 -> xyz=-0.201 0.1062 0.195 rpy=0.0 0.0 0.0
- joint base_antenna_right_joint: origin xyz=-0.201 -0.1062 0.195 rpy=0 0 0 -> xyz=-0.201 -0.1062 0.195 rpy=0.0 0.0 0.0
- joint base_footprint_joint: origin xyz=0 0 0.0985 rpy=0 0 0 -> xyz=0.0 0.0 0.0985 rpy=0.0 0.0 0.0
- joint base_imu_joint: origin xyz=0.10171 0 0.11282 rpy=0 0 -1.5707963267948966 -> xyz=0.10171 0.0 0.11282 rpy=0.0 0.0 -1.5707963267948966
- joint base_laser_joint: axis 0 1 0 -> 0.0 1.0 0.0; origin xyz=0.202 0.0 -0.004 rpy=0 0 0 -> xyz=0.202 0.0 -0.004 rpy=0.0 0.0 0.0
- joint base_mic_back_left_joint: origin xyz=-0.1082 -0.0599 0.195 rpy=0 0 0 -> xyz=-0.1082 -0.0599 0.195 rpy=0.0 0.0 0.0
- joint base_mic_back_right_joint: origin xyz=-0.1082 -0.13789 0.195 rpy=0 0 0 -> xyz=-0.1082 -0.13789 0.195 rpy=0.0 0.0 0.0
- joint base_mic_front_left_joint: origin xyz=0.23182 0.03902 0.195 rpy=0 0 0 -> xyz=0.23182 0.03902 0.195 rpy=0.0 0.0 0.0
- joint base_mic_front_right_joint: origin xyz=0.23182 -0.03902 0.195 rpy=0 0 0 -> xyz=0.23182 -0.03902 0.195 rpy=0.0 0.0 0.0
- joint base_sonar_01_joint: axis 0 0 1 -> 0.0 0.0 1.0; origin xyz=-0.183 -0.183 0.173 rpy=0 0 3.9269908169872414 -> xyz=-0.183 -0.183 0.173 rpy=0.0 0.0 3.9269908169872414
- joint base_sonar_02_joint: axis 0 0 1 -> 0.0 0.0 1.0; origin xyz=-0.259 0.0 0.173 rpy=0 0 3.141592653589793 -> xyz=-0.259 0.0 0.173 rpy=0.0 0.0 3.141592653589793
- joint base_sonar_03_joint: axis 0 0 1 -> 0.0 0.0 1.0; origin xyz=-0.183 0.183 0.173 rpy=0 0 2.356194490192345 -> xyz=-0.183 0.183 0.173 rpy=0.0 0.0 2.356194490192345
- joint caster_back_left_1_joint: axis 0 0 1 -> 0.0 0.0 1.0; origin xyz=-0.17350000000000002 0.102 -0.0335 rpy=0 0 0 -> xyz=-0.17350000000000002 0.102 -0.0335 rpy=0.0 0.0 0.0
- joint caster_back_left_2_joint: axis 0 0 1 -> 0.0 0.0 1.0; origin xyz=-0.016 0.0000 -0.040 rpy=-1.5707963267948966 0 0 -> xyz=-0.016 0.0 -0.04 rpy=-1.5707963267948966 0.0 0.0
- joint caster_back_right_1_joint: axis 0 0 1 -> 0.0 0.0 1.0; origin xyz=-0.17350000000000002 -0.102 -0.0335 rpy=0 0 0 -> xyz=-0.17350000000000002 -0.102 -0.0335 rpy=0.0 0.0 0.0
- joint caster_back_right_2_joint: axis 0 0 1 -> 0.0 0.0 1.0; origin xyz=-0.016 0.0000 -0.040 rpy=-1.5707963267948966 0 0 -> xyz=-0.016 0.0 -0.04 rpy=-1.5707963267948966 0.0 0.0
- joint caster_front_left_1_joint: axis 0 0 1 -> 0.0 0.0 1.0; origin xyz=0.1695 0.102 -0.0335 rpy=0 0 0 -> xyz=0.1695 0.102 -0.0335 rpy=0.0 0.0 0.0
- joint caster_front_left_2_joint: axis 0 0 1 -> 0.0 0.0 1.0; origin xyz=-0.016 0.0000 -0.040 rpy=-1.5707963267948966 0 0 -> xyz=-0.016 0.0 -0.04 rpy=-1.5707963267948966 0.0 0.0
- joint caster_front_right_1_joint: axis 0 0 1 -> 0.0 0.0 1.0; origin xyz=0.1695 -0.102 -0.0335 rpy=0 0 0 -> xyz=0.1695 -0.102 -0.0335 rpy=0.0 0.0 0.0
- joint caster_front_right_2_joint: axis 0 0 1 -> 0.0 0.0 1.0; origin xyz=-0.016 0.0000 -0.040 rpy=-1.5707963267948966 0 0 -> xyz=-0.016 0.0 -0.04 rpy=-1.5707963267948966 0.0 0.0
- joint cover_joint: origin xyz=0 0 0.13 rpy=0 0 0 -> xyz=0.0 0.0 0.13 rpy=0.0 0.0 0.0
- joint gripper_left_grasping_frame_joint: origin xyz=0 0 -0.12 rpy=-1.5708 1.5708 0 -> xyz=0.0 0.0 -0.12 rpy=-1.5708 1.5708 0.0
- joint gripper_left_joint: axis 0 0 0 -> 0.0 0.0 0.0; origin xyz=0.01 0 0 rpy=1.5707963267948966 1.5707963267948966 -1.5707963267948966 -> xyz=0.01 0.0 0.0 rpy=1.5707963267948966 1.5707963267948966 -1.5707963267948966
- joint gripper_left_left_finger_joint: axis -1 0 0 -> -1.0 0.0 0.0; limit lower=0 upper=0.045 effort=16 velocity=0.05 -> lower=0.0 upper=0.045 effort=16.0 velocity=0.05; origin xyz=0. 0 0 rpy=0 0 0 -> xyz=0.0 0.0 0.0 rpy=0.0 0.0 0.0
- joint gripper_left_right_finger_joint: axis 1 0 0 -> 1.0 0.0 0.0; limit lower=0.0 upper=0.045 effort=16 velocity=0.05 -> lower=0.0 upper=0.045 effort=16.0 velocity=0.05; origin xyz=0. 0 0 rpy=0 0 0 -> xyz=0.0 0.0 0.0 rpy=0.0 0.0 0.0
- joint gripper_left_tool_joint: axis 0 0 0 -> 0.0 0.0 0.0; origin xyz=0.01 0 0 rpy=1.5707963267948966 1.5707963267948966 -1.5707963267948966 -> xyz=0.01 0.0 0.0 rpy=1.5707963267948966 1.5707963267948966 -1.5707963267948966
- joint gripper_right_grasping_frame_joint: origin xyz=0 0 -0.12 rpy=-1.5708 1.5708 0 -> xyz=0.0 0.0 -0.12 rpy=-1.5708 1.5708 0.0
- joint gripper_right_joint: axis 0 0 0 -> 0.0 0.0 0.0; origin xyz=0.01 0 0 rpy=1.5707963267948966 1.5707963267948966 -1.5707963267948966 -> xyz=0.01 0.0 0.0 rpy=1.5707963267948966 1.5707963267948966 -1.5707963267948966
- joint gripper_right_left_finger_joint: axis -1 0 0 -> -1.0 0.0 0.0; limit lower=0 upper=0.045 effort=16 velocity=0.05 -> lower=0.0 upper=0.045 effort=16.0 velocity=0.05; origin xyz=0. 0 0 rpy=0 0 0 -> xyz=0.0 0.0 0.0 rpy=0.0 0.0 0.0
- joint gripper_right_right_finger_joint: axis 1 0 0 -> 1.0 0.0 0.0; limit lower=0.0 upper=0.045 effort=16 velocity=0.05 -> lower=0.0 upper=0.045 effort=16.0 velocity=0.05; origin xyz=0. 0 0 rpy=0 0 0 -> xyz=0.0 0.0 0.0 rpy=0.0 0.0 0.0
- joint gripper_right_tool_joint: axis 0 0 0 -> 0.0 0.0 0.0; origin xyz=0.01 0 0 rpy=1.5707963267948966 1.5707963267948966 -1.5707963267948966 -> xyz=0.01 0.0 0.0 rpy=1.5707963267948966 1.5707963267948966 -1.5707963267948966
- joint head_1_joint: axis 0 0 1 -> 0.0 0.0 1.0; origin xyz=0.182 0.0 0.0 rpy=0 0 0 -> xyz=0.182 0.0 0.0 rpy=0.0 0.0 0.0
- joint head_2_joint: axis 0 0 1 -> 0.0 0.0 1.0; origin xyz=0.005 0.0 0.098 rpy=1.5707963267948966 0 0 -> xyz=0.005 0.0 0.098 rpy=1.5707963267948966 0.0 0.0
- joint rgbd_laser_joint: origin xyz=-0.9 0 0 rpy=0 0 0 -> xyz=-0.9 0.0 0.0 rpy=0.0 0.0 0.0
- joint suspension_left_joint: axis 0 0 1 -> 0.0 0.0 1.0; origin xyz=0 0 0 rpy=0 0 0 -> xyz=0.0 0.0 0.0 rpy=0.0 0.0 0.0
- joint suspension_right_joint: axis 0 0 1 -> 0.0 0.0 1.0; origin xyz=0 0 0 rpy=0 0 0 -> xyz=0.0 0.0 0.0 rpy=0.0 0.0 0.0
- joint torso_fixed_column_joint: axis 0 0 0 -> 0.0 0.0 0.0; origin xyz=-0.062 0 0.195 rpy=0 0 0 -> xyz=-0.062 0.0 0.195 rpy=0.0 0.0 0.0
- joint torso_fixed_joint: axis 0 0 0 -> 0.0 0.0 0.0; origin xyz=-0.062 0.0 0.193 rpy=0 0 0 -> xyz=-0.062 0.0 0.193 rpy=0.0 0.0 0.0
- joint torso_lift_joint: axis 0 0 1 -> 0.0 0.0 1.0; limit lower=0 upper=0.35 effort=2000 velocity=0.07 -> lower=0.0 upper=0.35 effort=2000.0 velocity=0.07
- joint wheel_left_joint: axis 0 0 1 -> 0.0 0.0 1.0; limit effort=6.0 velocity=10.152284263959391 -> lower=0 upper=0 effort=6.0 velocity=10.152284263959391; origin xyz=0 0.2022 0.0 rpy=-1.5707963267948966 0 0 -> xyz=0.0 0.2022 0.0 rpy=-1.5707963267948966 0.0 0.0
- joint wheel_right_joint: axis 0 0 1 -> 0.0 0.0 1.0; limit effort=6.0 velocity=10.152284263959391 -> lower=0 upper=0 effort=6.0 velocity=10.152284263959391; origin xyz=0 -0.2022 0.0 rpy=-1.5707963267948966 0 0 -> xyz=0.0 -0.2022 0.0 rpy=-1.5707963267948966 0.0 0.0
- joint wrist_left_ft_joint: origin xyz=0.00785 0 0 rpy=1.5707963267948966 0 1.5707963267948966 -> xyz=0.00785 0.0 0.0 rpy=1.5707963267948966 0.0 1.5707963267948966
- joint wrist_left_tool_joint: origin xyz=0 0 0.012725 rpy=-1.5707963267948966 -1.5707963267948966 0 -> xyz=0.0 0.0 0.012725 rpy=-1.5707963267948966 -1.5707963267948966 0.0
- joint wrist_right_ft_joint: origin xyz=0.00785 0 0 rpy=1.5707963267948966 0 1.5707963267948966 -> xyz=0.00785 0.0 0.0 rpy=1.5707963267948966 0.0 1.5707963267948966
- joint wrist_right_tool_joint: origin xyz=0 0 0.012725 rpy=-1.5707963267948966 -1.5707963267948966 0 -> xyz=0.0 0.0 0.012725 rpy=-1.5707963267948966 -1.5707963267948966 0.0
- joint xtion_depth_joint: origin xyz=0.0 0.025 0.0 rpy=0 0 0 -> xyz=0.0 0.025 0.0 rpy=0.0 0.0 0.0
- joint xtion_depth_optical_joint: origin xyz=0 0 0 rpy=-1.5707963267948966 0.0 -1.5707963267948966 -> xyz=0.0 0.0 0.0 rpy=-1.5707963267948966 0.0 -1.5707963267948966
- joint xtion_optical_joint: origin xyz=0 0 0 rpy=-1.5707963267948966 0.0 -1.5707963267948966 -> xyz=0.0 0.0 0.0 rpy=-1.5707963267948966 0.0 -1.5707963267948966
- joint xtion_orbbec_aux_joint: origin xyz=0 0 0 rpy=0 0 0 -> xyz=0.0 0.0 0.0 rpy=0.0 0.0 0.0
- joint xtion_rgb_joint: origin xyz=0.0 0.022 0.0 rpy=0 0 0 -> xyz=0.0 0.022 0.0 rpy=0.0 0.0 0.0
- joint xtion_rgb_optical_joint: origin xyz=0 0 0 rpy=-1.5707963267948966 0.0 -1.5707963267948966 -> xyz=0.0 0.0 0.0 rpy=-1.5707963267948966 0.0 -1.5707963267948966

Commit message: Change gain + torsor limit

File: pal_robotics/tiago_dual_description/urdf/tiago_dual.urdf (robot description, URDF)
Before this commit: robot tiago_dual, 69 links, 68 joints
Joints:
- joint torso_lift_joint: limit lower=0.0 upper=0.35 effort=2000.0 velocity=0.07 -> lower=0.0 upper=2.00 effort=2000.0 velocity=0.07

Commit message: Fix limit

File: pal_robotics/tiago_dual_description/urdf/tiago_dual.urdf (robot description, URDF)
Before this commit: robot tiago_dual, 69 links, 68 joints
Joints:
- joint torso_lift_joint: limit lower=0.0 upper=2.00 effort=2000.0 velocity=0.07 -> lower=0.0 upper=0.8 effort=2000.0 velocity=0.07
